Commit message: Added right aileron

File: urdf/macros.xacro (robot description, xacro)
@@ -1,5 +1,5 @@
 <?xml version="1.0"?>
 <robot name="planesil" xmlns:xacro="http://www.ros.org/wiki/xacro">
-    <xacro:macro name="transmission" params= "joint_name">
+    <xacro:macro name="joint_transmission" params= "joint_name">
         <transmission name="${joint_name}_transmission">
             <type>transmission_interface/SimpleTransmission</type>

File: urdf/planesil_model.xacro (robot description, xacro)
@@ -58,15 +58,34 @@
         <limit lower="-0.5233" upper="0.5233" effort="100000" velocity="100000"/>
     </joint>
-    <!-- <xacro:transmission joint_name="left_aileron"/> -->
-    <transmission name="left_aileron_transmission">
-        <type>transmission_interface/SimpleTransmission</type>
-        <joint name="left_aileron_joint">
-            <hardwareInterface>hardware_interface/EffortJointInterface</hardwareInterface>
-        </joint>
-        <actuator name="left_aileron_servo">
-            <hardwareInterface>EffortJointInterface</hardwareInterface>
-            <mechanicalReduction>10</mechanicalReduction>
-        </actuator>
-    </transmission>
+    <xacro:joint_transmission joint_name="left_aileron"/>
+    <!-- Right aileron -->
+    <link name="right_aileron">
+        <inertial>
+            <origin xyz="1.85 3.7 -1.4" rpy="0.05 -0 -0.12" />
+            <mass value="2"/>
+            <inertia ixx="0.8434" ixy="0.0" ixz="0.0" iyy="0.0119" iyz="0.0" izz="0.855"/>
+        </inertial>
+        <collision>
+            <origin xyz="1.85 3.7 -1.4" rpy="0.05 -0 -0.12" />
+            <geometry>
+                <mesh filename="package://planesim_description/meshes/right_aileron.dae"/>
+            </geometry>
+        </collision>
+        <visual>
+            <origin xyz="1.85 3.7 -1.4" rpy="0.05 -0 -0.12" />
+            <geometry>
+                <mesh filename="package://planesim_description/meshes/right_aileron.dae"/>
+            </geometry>
+            <material name="blue"/>
+        </visual>
+    </link>
+    <joint name="right_aileron_joint" type="continuous">
+        <parent link="body"/>
+        <child link="right_aileron"/>
+        <axis xyz="0 1 0" rpy="0 0 0"/>
+        <origin xyz="-1.45 -3.7 1.5" rpy="-0.05 0 0.12" />
+        <limit lower="-0.5233" upper="0.5233" effort="100000" velocity="100000"/>
+    </joint>
+    <xacro:joint_transmission joint_name="right_aileron"/>
     <gazebo>
         <plugin name="gazebo_ros_control" filename="libgazebo_ros_control.so">

Commit message: Reworked model to start from scratch

File: urdf/macros.xacro (robot description, xacro)
@@ -1,4 +1,22 @@
 <?xml version="1.0"?>
 <robot name="planesil" xmlns:xacro="http://www.ros.org/wiki/xacro">
+    <macro name="cylinder_inertia" params="m r h">
+        <inertia  ixx="${m*(3*r*r+h*h)/12}" ixy = "0" ixz = "0"
+            iyy="${m*(3*r*r+h*h)/12}" iyz = "0"
+            izz="${m*r*r/2}"
+        />
+    </macro>
+    <macro name="box_inertia" params="m x y z">
+        <inertia  ixx="${m*(y*y+z*z)/12}" ixy = "0" ixz = "0"
+            iyy="${m*(x*x+z*z)/12}" iyz = "0"
+            izz="${m*(x*x+z*z)/12}"
+        />
+    </macro>
+    <macro name="sphere_inertia" params="m r">
+        <inertia  ixx="${2*m*r*r/5}" ixy = "0" ixz = "0"
+            iyy="${2*m*r*r/5}" iyz = "0"
+            izz="${2*m*r*r/5}"
+        />
+    </macro>
     <xacro:macro name="joint_transmission" params= "joint_name">
         <transmission name="${joint_name}_transmission">

File: urdf/planesil_model.xacro (robot description, xacro)
@@ -4,8 +4,7 @@
     <xacro:include filename="$(find planesim_description)/urdf/macros.xacro" />
     <!-- Body of plane -->
-    <link name="body">
+    <!-- <link name="body">
         <inertial>
             <origin xyz="-0.0414 0 0.9271" rpy="0 0 0"/>
-            <!-- <origin xyz="0 0 0" rpy="0 0 0"/> -->
             <mass value="680.389"/>
             <inertia ixx="1285.315427874" ixy="0.0" ixz="0.0" iyy="1824.930976707" iyz="0.0" izz="2666.893931043"/>
@@ -24,68 +23,73 @@
             <material name="blue"/>
         </visual>
+    </link> -->
+    <xacro:property name="bodyY" value="1"/>
+    <xacro:property name="bodyX" value="8"/>
+    <xacro:property name="bodyZ" value="1"/>
+    <xacro:property name="bodyMass" value="300"/>
+    <xacro:property name="wingY" value="5"/>
+    <xacro:property name="wingX" value="1.5"/>
+    <xacro:property name="wingZ" value="${bodyZ/2}"/>
+    <xacro:property name="wingMass" value="100"/>
+    <!-- X axis is down the runway -->
+    <link name="body">
+        <inertial>
+            <origin xyz="0 0 0" rpy="0 0 0"/>
+            <mass value="${bodyMass}"/>
+            <xacro:box_inertia m="${bodyMass}" x="${bodyX}" y="${bodyY}" z="${bodyZ}"/>
+        </inertial>
+        <collision>
+            <origin xyz="0 0 0" rpy="0 0 0"/>
+            <geometry>
+                <box size="${bodyX} ${bodyY} ${bodyZ}"/>
+            </geometry>
+        </collision>
+        <visual>
+            <origin xyz="0 0 0" rpy="0 0 0"/>
+            <geometry>
+                <box size="${bodyX} ${bodyY} ${bodyZ}"/>
+            </geometry>
+            <material name="orange"/>
+        </visual>
     </link>
-    <link name='base_link'/>
+    <gazebo reference="body">
+        <material>Gazebo/Orange</material>
+    </gazebo>
+    <link name="base_link"/>
     <joint name="base_joint" type="fixed">
         <parent link="base_link"/>
         <child link="body"/>
     </joint>
-    <!-- Left aileron -->
-    <link name="left_aileron">
+    <link name="leftWing">
         <inertial>
-            <origin xyz="1.85 -3.7 -1.4" rpy="-0.05 -0 0.12" />
-            <mass value="2"/>
-            <inertia ixx="0.8434" ixy="0.0" ixz="0.0" iyy="0.0119" iyz="0.0" izz="0.855"/>
+            <origin xyz="0 0 0" rpy="0 0 0"/>
+            <mass value="${wingMass}"/>
+            <xacro:box_inertia m="${wingMass}" x="${wingX}" y="${wingY}" z="${wingZ}"/>
         </inertial>
         <collision>
-            <origin xyz="1.85 -3.7 -1.4" rpy="-0.05 -0 0.12" />
+            <origin xyz="0 0 0" rpy="0 0 0"/>
             <geometry>
-                <mesh filename="package://planesim_description/meshes/left_aileron.dae"/>
+                <box size="${wingX} ${wingY} ${wingZ}"/>
             </geometry>
         </collision>
         <visual>
-            <origin xyz="1.85 -3.7 -1.4" rpy="-0.05 -0 0.12" />
+            <origin xyz="0 0 0" rpy="0 0 0"/>
             <geometry>
-                <mesh filename="package://planesim_description/meshes/left_aileron.dae"/>
+                <box size="${wingX} ${wingY} ${wingZ}"/>
             </geometry>
-            <material name="blue"/>
+            <material name="red"/>
         </visual>
     </link>
-    <joint name="left_aileron_joint" type="continuous">
+    <gazebo reference="leftWing">
+        <material>
+            Gazebo/Red
+        </material>
+    </gazebo>
+    <joint name="leftWing_joint" type="continuous">
         <parent link="body"/>
-        <child link="left_aileron"/>
+        <child link="leftWing"/>
+        <origin xyz="0 ${bodyY/2 + wingY/2} 0" rpy="0 0 0"/>
         <axis xyz="0 1 0" rpy="0 0 0"/>
-        <origin xyz="-1.45 3.7 1.5" rpy="0.05 0 -0.12" />
-        <limit lower="-0.5233" upper="0.5233" effort="100000" velocity="100000"/>
     </joint>
-    <xacro:joint_transmission joint_name="left_aileron"/>
-    <!-- Right aileron -->
-    <link name="right_aileron">
-        <inertial>
-            <origin xyz="1.85 3.7 -1.4" rpy="0.05 -0 -0.12" />
-            <mass value="2"/>
-            <inertia ixx="0.8434" ixy="0.0" ixz="0.0" iyy="0.0119" iyz="0.0" izz="0.855"/>
-        </inertial>
-        <collision>
-            <origin xyz="1.85 3.7 -1.4" rpy="0.05 -0 -0.12" />
-            <geometry>
-                <mesh filename="package://planesim_description/meshes/right_aileron.dae"/>
-            </geometry>
-        </collision>
-        <visual>
-            <origin xyz="1.85 3.7 -1.4" rpy="0.05 -0 -0.12" />
-            <geometry>
-                <mesh filename="package://planesim_description/meshes/right_aileron.dae"/>
-            </geometry>
-            <material name="blue"/>
-        </visual>
-    </link>
-    <joint name="right_aileron_joint" type="continuous">
-        <parent link="body"/>
-        <child link="right_aileron"/>
-        <axis xyz="0 1 0" rpy="0 0 0"/>
-        <origin xyz="-1.45 -3.7 1.5" rpy="-0.05 0 0.12" />
-        <limit lower="-0.5233" upper="0.5233" effort="100000" velocity="100000"/>
-    </joint>
-    <xacro:joint_transmission joint_name="right_aileron"/>
     <gazebo>
         <plugin name="gazebo_ros_control" filename="libgazebo_ros_control.so">

Commit message: Added wheels

File: urdf/macros.xacro (robot description, xacro)
@@ -31,4 +31,42 @@
         </transmission>
     </xacro:macro>
+    <xacro:macro name="wheel" params="name front left">
+         <link name="${name}_wheel">
+            <collision>
+                <origin xyz="0 0 0" rpy="0 ${PI/2} ${PI/2}" />
+                <geometry>
+                <cylinder length="${wheelWidth}" radius="${wheelRadius}"/>
+                </geometry>
+            </collision>
+            <visual>
+                <origin xyz="0 0 0" rpy="0 ${PI/2} ${PI/2}" />
+                <geometry>
+                <cylinder length="${wheelWidth}" radius="${wheelRadius}"/>
+                </geometry>
+                <material name="black"/>
+            </visual>
+            <inertial>
+                <origin xyz="0 0 0" rpy="0 ${PI/2} ${PI/2}" />
+                <mass value="${wheelMass}"/>
+                <xacro:cylinder_inertia m="${wheelMass}" r="${wheelRadius}" h="${wheelWidth}"/>
+            </inertial>
+        </link>
+        <gazebo reference="${name}_wheel">
+            <mu1 value="1.0"/>
+            <mu2 value="1.0"/>
+            <kp  value="10000000.0" />
+            <kd  value="1.0" />
+            <fdir1 value="1 0 0"/>
+            <material>Gazebo/Black</material>
+        </gazebo>
+        <joint name="${name}_wheel_hinge" type="continuous">
+            <parent link="body"/>
+            <child link="${name}_wheel"/>
+            <origin xyz="${front * (bodyX/2 - wheelRadius)} ${left * (bodyY/2 + wheelWidth/2)} ${-bodyZ/2}" rpy="0 0 0" />
+            <axis xyz="0 1 0" rpy="0 0 0" />
+            <limit effort="100" velocity="100"/>
+            <joint_properties damping="0.0" friction="0.5"/>
+        </joint>
+    </xacro:macro>
 <!--
 xacro template:

File: urdf/planesil_model.xacro (robot description, xacro)
@@ -24,7 +24,8 @@
         </visual>
     </link> -->
-    <xacro:property name="bodyY" value="1"/>
+    <xacro:property name="PI" value="3.14"/>
+    <xacro:property name="bodyY" value="0.5"/>
     <xacro:property name="bodyX" value="8"/>
-    <xacro:property name="bodyZ" value="1"/>
+    <xacro:property name="bodyZ" value="0.5"/>
     <xacro:property name="bodyMass" value="300"/>
     <xacro:property name="wingY" value="5"/>
@@ -32,4 +33,7 @@
     <xacro:property name="wingZ" value="${bodyZ/4}"/>
     <xacro:property name="wingMass" value="100"/>
+    <xacro:property name="wheelWidth" value="0.1"/>
+    <xacro:property name="wheelRadius" value="0.5"/>
+    <xacro:property name="wheelMass" value="5"/>
     <!-- X axis is down the runway -->
     <link name="body">
@@ -123,4 +127,8 @@
         <axis xyz="0 1 0" rpy="0 0 0"/>
     </joint>
+    <xacro:wheel name="frontLeft_wheel" front="1" left="1" />
+    <xacro:wheel name="frontRight_wheel" front="1" left="-1" />
+    <xacro:wheel name="backLeft_wheel" front="-1" left="1" />
+    <xacro:wheel name="backRight_wheel" front="-1" left="-1" />
     <gazebo>
         <plugin name="gazebo_ros_control" filename="libgazebo_ros_control.so">

Commit message: Added landing gear link

File: urdf/macros.xacro (robot description, xacro)
@@ -30,4 +30,59 @@
             </actuator>
         </transmission>
+    </xacro:macro>
+    <xacro:macro name="wing" params="name left">
+        <link name="${name}_wing">
+            <inertial>
+                <origin xyz="0 0 0" rpy="0 0 0"/>
+                <mass value="${wingMass}"/>
+                <xacro:box_inertia m="${wingMass}" x="${wingX}" y="${wingY}" z="${wingZ}"/>
+            </inertial>
+            <collision>
+                <origin xyz="0 0 0" rpy="0 0 0"/>
+                <geometry>
+                    <box size="${wingX} ${wingY} ${wingZ}"/>
+                </geometry>
+            </collision>
+            <visual>
+                <origin xyz="0 0 0" rpy="0 0 0"/>
+                <geometry>
+                    <box size="${wingX} ${wingY} ${wingZ}"/>
+                </geometry>
+                <material name="red"/>
+            </visual>
+        </link>
+        <joint name="${name}_wing_joint" type="continuous">
+            <parent link="body"/>
+            <child link="${name}_wing"/>
+            <origin xyz="0 ${left * (bodyY/2 + wingY/2)} 0" rpy="0 0 0"/>
+            <axis xyz="0 1 0" rpy="0 0 0"/>
+        </joint>
+    </xacro:macro>
+    <xacro:macro name="landingGear" params="name front">
+        <link name="${name}_landingGear">
+            <inertial>
+                <origin xyz="0 0 0" rpy="0 0 0"/>
+                <mass value="${landingGearMass}"/>
+                <xacro:box_inertia m="${landingGearMass}" x="${landingGearX}" y="${landingGearY}" z="${landingGearZ}"/>
+            </inertial>
+            <collision>
+                <origin xyz="0 0 0" rpy="0 0 0"/>
+                <geometry>
+                    <box size="${landingGearX} ${landingGearY} ${landingGearZ}"/>
+                </geometry>
+            </collision>
+            <visual>
+                <origin xyz="0 0 0" rpy="0 0 0"/>
+                <geometry>
+                    <box size="${landingGearX} ${landingGearY} ${landingGearZ}"/>
+                </geometry>
+                <material name="orange"/>
+            </visual>
+        </link>
+        <joint name="${name}_landingGear_joint" type="fixed">
+            <parent link="body"/>
+            <child link="${name}_landingGear"/>
+            <origin xyz="${front * (bodyX/2 - landingGearX/2)} 0 ${bodyZ/2-landingGearZ/2}" rpy="0 0 0"/>
+        </joint>
     </xacro:macro>
     <xacro:macro name="wheel" params="name front left">

File: urdf/planesil_model.xacro (robot description, xacro)
@@ -26,13 +26,17 @@
     <xacro:property name="PI" value="3.14"/>
     <xacro:property name="bodyY" value="0.5"/>
-    <xacro:property name="bodyX" value="8"/>
+    <xacro:property name="bodyX" value="6"/>
     <xacro:property name="bodyZ" value="0.5"/>
     <xacro:property name="bodyMass" value="300"/>
     <xacro:property name="wingY" value="5"/>
-    <xacro:property name="wingX" value="1.5"/>
+    <xacro:property name="wingX" value="1"/>
     <xacro:property name="wingZ" value="${bodyZ/4}"/>
     <xacro:property name="wingMass" value="100"/>
+    <xacro:property name="landingGearY" value="${bodyY}"/>
+    <xacro:property name="landingGearX" value="0.125"/>
+    <xacro:property name="landingGearZ" value="1"/>
+    <xacro:property name="landingGearMass" value="10"/>
     <xacro:property name="wheelWidth" value="0.1"/>
-    <xacro:property name="wheelRadius" value="0.5"/>
+    <xacro:property name="wheelRadius" value="0.25"/>
     <xacro:property name="wheelMass" value="5"/>
     <!-- X axis is down the runway -->
@@ -65,66 +69,16 @@
         <child link="body"/>
     </joint>
-    <link name="leftWing">
-        <inertial>
-            <origin xyz="0 0 0" rpy="0 0 0"/>
-            <mass value="${wingMass}"/>
-            <xacro:box_inertia m="${wingMass}" x="${wingX}" y="${wingY}" z="${wingZ}"/>
-        </inertial>
-        <collision>
-            <origin xyz="0 0 0" rpy="0 0 0"/>
-            <geometry>
-                <box size="${wingX} ${wingY} ${wingZ}"/>
-            </geometry>
-        </collision>
-        <visual>
-            <origin xyz="0 0 0" rpy="0 0 0"/>
-            <geometry>
-                <box size="${wingX} ${wingY} ${wingZ}"/>
-            </geometry>
-            <material name="red"/>
-        </visual>
-    </link>
-    <gazebo reference="leftWing">
+    <xacro:wing name="left" left="1"/>
+    <gazebo reference="left_wing">
         <material>
             Gazebo/Red
         </material>
     </gazebo>
-    <joint name="leftWing_joint" type="continuous">
-        <parent link="body"/>
-        <child link="leftWing"/>
-        <origin xyz="0 ${bodyY/2 + wingY/2} 0" rpy="0 0 0"/>
-        <axis xyz="0 1 0" rpy="0 0 0"/>
-    </joint>
-    <link name="rightWing">
-        <inertial>
-            <origin xyz="0 0 0" rpy="0 0 0"/>
-            <mass value="${wingMass}"/>
-            <xacro:box_inertia m="${wingMass}" x="${wingX}" y="${wingY}" z="${wingZ}"/>
-        </inertial>
-        <collision>
-            <origin xyz="0 0 0" rpy="0 0 0"/>
-            <geometry>
-                <box size="${wingX} ${wingY} ${wingZ}"/>
-            </geometry>
-        </collision>
-        <visual>
-            <origin xyz="0 0 0" rpy="0 0 0"/>
-            <geometry>
-                <box size="${wingX} ${wingY} ${wingZ}"/>
-            </geometry>
-            <material name="green"/>
-        </visual>
-    </link>
-    <gazebo reference="rightWing">
+    <xacro:wing name="right" left="-1"/>
+    <gazebo reference="right_wing">
         <material>
             Gazebo/Green
         </material>
     </gazebo>
-    <joint name="rightWing_joint" type="continuous">
-        <parent link="body"/>
-        <child link="rightWing"/>
-        <origin xyz="0 ${-(bodyY/2 + wingY/2)} 0" rpy="0 0 0"/>
-        <axis xyz="0 1 0" rpy="0 0 0"/>
-    </joint>
     <xacro:wheel name="frontLeft_wheel" front="1" left="1" />
     <xacro:wheel name="frontRight_wheel" front="1" left="-1" />

Commit message: Joined wheels to landingGear

File: urdf/macros.xacro (robot description, xacro)
@@ -116,7 +116,12 @@
         </gazebo>
         <joint name="${name}_wheel_hinge" type="continuous">
-            <parent link="body"/>
+            <xacro:if value="${front == 1}">
+                <parent link="front_landingGear"/>
+            </xacro:if>
+            <xacro:unless value="${front == 1}">
+                <parent link="back_landingGear"/>
+            </xacro:unless>
             <child link="${name}_wheel"/>
-            <origin xyz="${front * (bodyX/2 - wheelRadius)} ${left * (bodyY/2 + wheelWidth/2)} ${-bodyZ/2}" rpy="0 0 0" />
+            <origin xyz="0 ${left * (landingGearY/2 + wheelWidth/2)} ${-landingGearZ/2}" rpy="0 0 0" />
             <axis xyz="0 1 0" rpy="0 0 0" />
             <limit effort="100" velocity="100"/>

File: urdf/planesil_model.xacro (robot description, xacro)
@@ -81,4 +81,6 @@
         </material>
     </gazebo>
+    <xacro:landingGear name="front" front="1"/>
+    <xacro:landingGear name="back" front="-1"/>
     <xacro:wheel name="frontLeft_wheel" front="1" left="1" />
     <xacro:wheel name="frontRight_wheel" front="1" left="-1" />

Commit message: Conditional wing colors for port/starboard

File: urdf/macros.xacro (robot description, xacro)
@@ -49,7 +49,25 @@
                     <box size="${wingX} ${wingY} ${wingZ}"/>
                 </geometry>
-                <material name="red"/>
+                <!-- Port/Starboard colors -->
+                <xacro:if value="${left == 1}">
+                    <material name="red"/>
+                </xacro:if>
+                <xacro:unless value="${left == 1}">
+                    <material name="green"/>
+                </xacro:unless>
             </visual>
         </link>
+        <gazebo reference="${name}_wing">
+            <xacro:if value="${left == 1}">
+                <material>
+                    Gazebo/Red
+                </material>
+            </xacro:if>
+            <xacro:unless value="${left == 1}">
+                <material>
+                    Gazebo/Green
+                </material>
+            </xacro:unless>
+        </gazebo>
         <joint name="${name}_wing_joint" type="continuous">
             <parent link="body"/>
@@ -116,4 +134,5 @@
         </gazebo>
         <joint name="${name}_wheel_hinge" type="continuous">
+            <!-- Different parent landingGears for front/back wheels -->
             <xacro:if value="${front == 1}">
                 <parent link="front_landingGear"/>

File: urdf/planesil_model.xacro (robot description, xacro)
@@ -70,15 +70,5 @@
     </joint>
     <xacro:wing name="left" left="1"/>
-    <gazebo reference="left_wing">
-        <material>
-            Gazebo/Red
-        </material>
-    </gazebo>
     <xacro:wing name="right" left="-1"/>
-    <gazebo reference="right_wing">
-        <material>
-            Gazebo/Green
-        </material>
-    </gazebo>
     <xacro:landingGear name="front" front="1"/>
     <xacro:landingGear name="back" front="-1"/>
