Commit message: Added propellor and propellorblock

File: urdf/macros.xacro (robot description, xacro)
@@ -98,4 +98,7 @@
             </visual>
         </link>
+        <gazebo reference="${name}_landingGear">
+            <material>Gazebo/Orange</material>
+        </gazebo>
         <joint name="${name}_landingGear_joint" type="fixed">
             <parent link="body"/>
@@ -148,4 +151,34 @@
         </joint>
     </xacro:macro>
+    <!-- <xacro:macro name="propellorBlade" params="name top">
+        <link name="${name}_propellorBlade">
+            <inertial>
+                <origin xyz="0 0 ${top * propellorBladeX/2}" rpy="0 ${PI/2} 0"/>
+                <mass value="${propellorBladeMass}"/>
+                <xacro:box_inertia m="${propellorBladeMass}" x="${propellorBladeX}" y="${propellorBladeY}" z="${propellorBladeZ}"/>
+            </inertial>
+            <collision>
+                <origin xyz="0 0 ${top * propellorBladeX/2}" rpy="0 ${PI/2} 0"/>
+                <geometry>
+                    <box size="${propellorBladeX} ${propellorBladeY} ${propellorBladeZ}"/>
+                </geometry>
+            </collision>
+            <visual>
+                <origin xyz="0 0 ${top * propellorBladeX/2}" rpy="0 ${PI/2} 0"/>
+                <geometry>
+                    <box size="${propellorBladeX} ${propellorBladeY} ${propellorBladeZ}"/>
+                </geometry>
+                <material name="blue"/>
+            </visual>
+        </link>
+        <gazebo reference="${name}_propellorBlade">
+            <material>Gazebo/Blue</material>
+        </gazebo>
+        <joint name="${name}_propellorBlade_joint" type="continuous">
+            <parent link="propellorBlock"/>
+            <child link="${name}_propellorBlade"/>
+            <origin xyz="${propellorBlockX/2 + propellorBladeZ/2} 0 0" rpy="0 0 0" />
+        </joint>
+    </xacro:macro> -->
 <!--
 xacro template:

File: urdf/planesil_model.xacro (robot description, xacro)
@@ -3,25 +3,4 @@
     <xacro:include filename="$(find planesim_description)/urdf/materials.xacro" />
     <xacro:include filename="$(find planesim_description)/urdf/macros.xacro" />
-    <!-- Body of plane -->
-    <!-- <link name="body">
-        <inertial>
-            <origin xyz="-0.0414 0 0.9271" rpy="0 0 0"/>
-            <mass value="680.389"/>
-            <inertia ixx="1285.315427874" ixy="0.0" ixz="0.0" iyy="1824.930976707" iyz="0.0" izz="2666.893931043"/>
-        </inertial>
-        <collision>
-            <origin xyz="0 0 0" rpy="0 0 0"/>
-            <geometry>
-                <mesh filename="package://planesim_description/meshes/body.dae"/>
-            </geometry>
-        </collision>
-        <visual>
-            <origin xyz="0 0 0" rpy="0 0 0"/>
-            <geometry>
-                <mesh filename="package://planesim_description/meshes/body.dae"/>
-            </geometry>
-            <material name="blue"/>
-        </visual>
-    </link> -->
     <xacro:property name="PI" value="3.14"/>
     <xacro:property name="bodyY" value="0.5"/>
@@ -40,5 +19,15 @@
     <xacro:property name="wheelRadius" value="0.25"/>
     <xacro:property name="wheelMass" value="5"/>
+    <xacro:property name="propellorBlockX" value="0.25"/>
+    <xacro:property name="propellorBlockY" value="${bodyY/2}"/>
+    <xacro:property name="propellorBlockZ" value="${bodyZ/2}" />
+    <xacro:property name="propellorBlockMass" value="5"/>
+    <xacro:property name="propellorX" value="1.5"/>      <!-- Length of blade -->
+    <xacro:property name="propellorY" value="0.2"/>   <!-- Width of blade -->
+    <xacro:property name="propellorZ" value="0.1"/>    <!-- Thickness of blade -->
+    <xacro:property name="propellorMass" value="2"/>
     <!-- X axis is down the runway -->
+    <!-- Y axis is to the left of the runway, looking down -->
+    <!-- Z axis is up -->
     <link name="body">
         <inertial>
@@ -77,4 +66,60 @@
     <xacro:wheel name="backLeft_wheel" front="-1" left="1" />
     <xacro:wheel name="backRight_wheel" front="-1" left="-1" />
+    <link name="propellorBlock">
+        <inertial>
+            <origin xyz="0 0 0" rpy="0 0 0"/>
+            <mass value="${propellorBlockMass}"/>
+            <xacro:box_inertia m="${propellorBlockMass}" x="${propellorBlockX}" y="${propellorBlockY}" z="${propellorBlockZ}"/>
+        </inertial>
+        <collision>
+            <origin xyz="0 0 0" rpy="0 0 0"/>
+            <geometry>
+                <box size="${propellorBlockX} ${propellorBlockY} ${propellorBlockZ}"/>
+            </geometry>
+        </collision>
+        <visual>
+            <origin xyz="0 0 0" rpy="0 0 0"/>
+            <geometry>
+                <box size="${propellorBlockX} ${propellorBlockY} ${propellorBlockZ}"/>
+            </geometry>
+            <material name="orange"/>
+        </visual>
+    </link>
+    <gazebo reference="propellorBlock">
+        <material>Gazebo/Orange</material>
+    </gazebo>
+    <joint name="propellorBlockJoint" type="fixed">
+        <parent link="body"/>
+        <child link="propellorBlock"/>
+        <origin xyz="${bodyX/2 + propellorBlockX/2} 0 0" rpy="0 0 0"/>
+    </joint>
+    <link name="propellor">
+        <inertial>
+            <origin xyz="0 0 0" rpy="0 ${PI/2} 0"/>
+            <mass value="${propellorMass}"/>
+            <xacro:box_inertia m="${propellorMass}" x="${propellorX}" y="${propellorY}" z="${propellorZ}"/>
+        </inertial>
+        <collision>
+            <origin xyz="0 0 0" rpy="0 ${PI/2} 0"/>
+            <geometry>
+                <box size="${propellorX} ${propellorY} ${propellorZ}"/>
+            </geometry>
+        </collision>
+        <visual>
+            <origin xyz="0 0 0" rpy="0 ${PI/2} 0"/>
+            <geometry>
+                <box size="${propellorX} ${propellorY} ${propellorZ}"/>
+            </geometry>
+            <material name="blue"/>
+        </visual>
+    </link>
+    <gazebo reference="propellor">
+        <material>Gazebo/Blue</material>
+    </gazebo>
+    <joint name="propellorJoint" type="continuous">
+        <parent link="propellorBlock" />
+        <child link="propellor" />
+        <origin xyz="${propellorBlockX/2 + propellorZ/2} 0 0" rpy="0 0 0"/>
+    </joint>
     <gazebo>
         <plugin name="gazebo_ros_control" filename="libgazebo_ros_control.so">

Commit message: removed extra prop blade macro

File: urdf/macros.xacro (robot description, xacro)
@@ -151,34 +151,4 @@
         </joint>
     </xacro:macro>
-    <!-- <xacro:macro name="propellorBlade" params="name top">
-        <link name="${name}_propellorBlade">
-            <inertial>
-                <origin xyz="0 0 ${top * propellorBladeX/2}" rpy="0 ${PI/2} 0"/>
-                <mass value="${propellorBladeMass}"/>
-                <xacro:box_inertia m="${propellorBladeMass}" x="${propellorBladeX}" y="${propellorBladeY}" z="${propellorBladeZ}"/>
-            </inertial>
-            <collision>
-                <origin xyz="0 0 ${top * propellorBladeX/2}" rpy="0 ${PI/2} 0"/>
-                <geometry>
-                    <box size="${propellorBladeX} ${propellorBladeY} ${propellorBladeZ}"/>
-                </geometry>
-            </collision>
-            <visual>
-                <origin xyz="0 0 ${top * propellorBladeX/2}" rpy="0 ${PI/2} 0"/>
-                <geometry>
-                    <box size="${propellorBladeX} ${propellorBladeY} ${propellorBladeZ}"/>
-                </geometry>
-                <material name="blue"/>
-            </visual>
-        </link>
-        <gazebo reference="${name}_propellorBlade">
-            <material>Gazebo/Blue</material>
-        </gazebo>
-        <joint name="${name}_propellorBlade_joint" type="continuous">
-            <parent link="propellorBlock"/>
-            <child link="${name}_propellorBlade"/>
-            <origin xyz="${propellorBlockX/2 + propellorBladeZ/2} 0 0" rpy="0 0 0" />
-        </joint>
-    </xacro:macro> -->
 <!--
 xacro template:

Commit message: Wing mechanical reduction

File: urdf/macros.xacro (robot description, xacro)
@@ -19,5 +19,5 @@
         />
     </macro>
-    <xacro:macro name="joint_transmission" params= "joint_name">
+    <xacro:macro name="joint_transmission" params= "joint_name reduction:=10">
         <transmission name="${joint_name}_transmission">
             <type>transmission_interface/SimpleTransmission</type>
@@ -27,5 +27,5 @@
             <actuator name="${joint_name}_servo">
                 <hardwareInterface>EffortJointInterface</hardwareInterface>
-                <mechanicalReduction>10</mechanicalReduction>
+                <mechanicalReduction>${reduction}</mechanicalReduction>
             </actuator>
         </transmission>
@@ -76,5 +76,5 @@
             <axis xyz="0 1 0" rpy="0 0 0"/>
         </joint>
-        <xacro:joint_transmission joint_name="${name}_wing" />
+        <xacro:joint_transmission joint_name="${name}_wing" reduction="100" />
     </xacro:macro>
     <xacro:macro name="landingGear" params="name front">

File: urdf/planesil_model.xacro (robot description, xacro)
@@ -160,5 +160,4 @@
             <link_name>propeller</link_name>
         </plugin>
-<!--
         <plugin name="leftWing" filename="libLiftDragPlugin.so">
             <a0>0.05984281113</a0>
@@ -171,5 +170,5 @@
             <cma_stall>0</cma_stall>
             <air_density> 1.2041 </air_density>
-            <cp> ${wingX/2} ${wingY/2} ${wingZ/2}</cp>
+            <cp> ${wingX/2} ${wingY/2} 0</cp>
             <area> ${(wingX/2) * (wingY/2)}</area>
             <forward> 1 0 0 </forward>
@@ -187,11 +186,11 @@
             <cma_stall>0</cma_stall>
             <air_density> 1.2041 </air_density>
-            <cp> ${wingX/2} ${wingY/2} ${wingZ/2}</cp>
+            <cp> ${wingX/2} ${wingY/2} 0</cp>
             <area> ${(wingX/2) * (wingY/2)}</area>
             <forward> 1 0 0 </forward>
             <upward> 0 0 1 </upward>
-            <link_name>left_wing</link_name>
-        </plugin>
-        <controller:gazebo_ros_imu name="imu_controller" plugin="libgazebo_ros_imu.so">
+            <link_name>right_wing</link_name>
+        </plugin>
+        <!-- <controller:gazebo_ros_imu name="imu_controller" plugin="libgazebo_ros_imu.so">
             <alwaysOn>true</alwaysOn>
             <updateRate>50.0</updateRate>
@@ -202,6 +201,5 @@
             <rpyOffsets>0 0 0</rpyOffsets>
             <interface:position name="imu_position"/>
-        </controller:gazebo_ros_imu>
-         -->
+        </controller:gazebo_ros_imu> -->
     </gazebo>
     <xacro:property name="counterWeightCoGXOffset" value="${((propellerBlockMass * propellerBlockX/2) + propellerMass * (propellerBlockX/2 + propellerZ/2))

Commit message: made plane wing joint fixed

File: urdf/macros.xacro (robot description, xacro)
@@ -70,11 +70,9 @@
             </xacro:unless>
         </gazebo>
-        <joint name="${name}_wing_joint" type="continuous">
+        <joint name="${name}_wing_joint" type="fixed">
             <parent link="body"/>
             <child link="${name}_wing"/>
             <origin xyz="0 ${left * (bodyY/2 + wingY/2)} 0" rpy="0 0 0"/>
-            <axis xyz="0 1 0" rpy="0 0 0"/>
         </joint>
-        <xacro:joint_transmission joint_name="${name}_wing" reduction="100" />
     </xacro:macro>
     <xacro:macro name="landingGear" params="name front">

Commit message: Oops nvm

File: urdf/macros.xacro (robot description, xacro)
@@ -70,9 +70,11 @@
             </xacro:unless>
         </gazebo>
-        <joint name="${name}_wing_joint" type="fixed">
+        <joint name="${name}_wing_joint" type="continuous">
             <parent link="body"/>
             <child link="${name}_wing"/>
             <origin xyz="0 ${left * (bodyY/2 + wingY/2)} 0" rpy="0 0 0"/>
+            <axis xyz="0 1 0" rpy="0 0 0"/>
         </joint>
+        <xacro:joint_transmission joint_name="${name}_wing" reduction="100" />
     </xacro:macro>
     <xacro:macro name="landingGear" params="name front">

Commit message: Added customLiftDrag, changed wing to use ailerons

File: urdf/macros.xacro (robot description, xacro)
@@ -70,5 +70,5 @@
             </xacro:unless>
         </gazebo>
-        <joint name="${name}_wing_joint" type="continuous">
+        <joint name="${name}_wing_joint" type="fixed">
             <parent link="body"/>
             <child link="${name}_wing"/>
@@ -76,5 +76,37 @@
             <axis xyz="0 1 0" rpy="0 0 0"/>
         </joint>
-        <xacro:joint_transmission joint_name="${name}_wing" reduction="100" />
+        <link name="${name}_aileron">
+            <inertial>
+                <origin xyz="0 0 0" rpy="0 0 0"/>
+                <mass value="${wingMass/5}"/>
+                <xacro:box_inertia m="${wingMass/5}" x="${wingX/5}" y="${wingY}" z="${wingZ}"/>
+            </inertial>
+            <collision>
+                <origin xyz="0 0 0" rpy="0 0 0"/>
+                <geometry>
+                    <box size="${wingX/5} ${wingY} ${wingZ}"/>
+                </geometry>
+            </collision>
+            <visual>
+                <origin xyz="0 0 0" rpy="0 0 0"/>
+                <geometry>
+                    <box size="${wingX/5} ${wingY} ${wingZ}"/>
+                </geometry>
+                <!-- Port/Starboard colors -->
+                <xacro:if value="${left == 1}">
+                    <material name="red"/>
+                </xacro:if>
+                <xacro:unless value="${left == 1}">
+                    <material name="green"/>
+                </xacro:unless>
+            </visual>
+        </link>
+        <joint name="${name}_aileron_joint" type="continuous">
+            <parent link="${name}_wing" />
+            <child link="${name}_aileron" />
+            <origin xyz="${-wingX/2 + -wingX/10} 0 0" rpy="0 0 0" />
+            <axis xyz="0 1 0" rpy="0 0 0" />
+        </joint>
+        <joint_transmission joint_name="${name}_aileron" reduction="100"/>
     </xacro:macro>
     <xacro:macro name="landingGear" params="name front">

File: urdf/planesil_model.xacro (robot description, xacro)
@@ -51,5 +51,5 @@
     </link>
     <gazebo reference="body">
-        <material>Gazebo/Orange</material>
+        <material>Gazebo/Gray</material>
     </gazebo>
     <link name="base_link"/>
@@ -127,4 +127,37 @@
     </joint>
     <xacro:joint_transmission joint_name="propeller"/>
+    <link name="leftWingCP">
+        <visual>
+            <origin xyz="0 0 0" rpy="0 0 0"/>
+            <geometry>
+                <sphere radius="0.1"/>
+            </geometry>
+            <material name="orange"/>
+        </visual>
+    </link>
+    <gazebo reference="leftWingCP">
+        <material>Gazebo/Orange</material>
+    </gazebo>
+    <joint name="leftWingCP_joint" type="fixed">
+        <parent link="body"/>
+        <child link="leftWingCP"/>
+        <origin xyz="0 ${wingY/2} ${wingZ/2}" rpy="0 0 0"/>
+    </joint>
+    <link name="rightWingCP">
+        <visual>
+            <origin xyz="0 ${-wingY/2} ${wingZ/2}" rpy="0 0 0"/>
+            <geometry>
+                <sphere radius="0.1"/>
+            </geometry>
+            <material name="orange"/>
+        </visual>
+    </link>
+    <gazebo reference="rightWingCP">
+        <material>Gazebo/Orange</material>
+    </gazebo>
+    <joint name="rightWingCP_joint" type="fixed">
+        <parent link="base_link"/>
+        <child link="rightWingCP"/>
+    </joint>
     <gazebo>
         <plugin name="propellerTopBlade" filename="libLiftDragPlugin.so">
@@ -160,5 +193,5 @@
             <link_name>propeller</link_name>
         </plugin>
-        <plugin name="leftWing" filename="libLiftDragPlugin.so">
+        <plugin name="leftWing" filename="libplanesim_liftdrag.so">
             <a0>0.05984281113</a0>
             <cla>4.752798721</cla>
@@ -170,11 +203,13 @@
             <cma_stall>0</cma_stall>
             <air_density> 1.2041 </air_density>
-            <cp> ${wingX/2} ${wingY/2} 0</cp>
+            <cp> 0 ${wingY/2} ${wingZ/2}</cp>
             <area> ${(wingX/2) * (wingY/2)}</area>
             <forward> 1 0 0 </forward>
             <upward> 0 0 1 </upward>
-            <link_name>left_wing</link_name>
-        </plugin>
-        <plugin name="rightWing" filename="libLiftDragPlugin.so">
+            <link_name>base_link</link_name>
+            <control_joint_name>left_aileron_joint</control_joint_name>
+            <control_joint_rad_to_cl>-2.0</control_joint_rad_to_cl>
+        </plugin>
+        <plugin name="rightWing" filename="libplanesim_liftdrag.so">
             <a0>0.05984281113</a0>
             <cla>4.752798721</cla>
@@ -186,9 +221,11 @@
             <cma_stall>0</cma_stall>
             <air_density> 1.2041 </air_density>
-            <cp> ${wingX/2} ${wingY/2} 0</cp>
+            <cp> 0 ${-wingY/2} ${wingZ/2}</cp>
             <area> ${(wingX/2) * (wingY/2)}</area>
             <forward> 1 0 0 </forward>
             <upward> 0 0 1 </upward>
-            <link_name>right_wing</link_name>
+            <link_name>base_link</link_name>
+            <control_joint_name>right_aileron_joint</control_joint_name>
+            <control_joint_rad_to_cl>-2.0</control_joint_rad_to_cl>
         </plugin>
         <!-- <controller:gazebo_ros_imu name="imu_controller" plugin="libgazebo_ros_imu.so">

Commit message: Changed CP markers to macro

File: urdf/macros.xacro (robot description, xacro)
@@ -19,5 +19,5 @@
         />
     </macro>
-    <xacro:macro name="joint_transmission" params= "joint_name reduction:=10">
+    <xacro:macro name="joint_transmission" params="joint_name reduction:=10">
         <transmission name="${joint_name}_transmission">
             <type>transmission_interface/SimpleTransmission</type>
@@ -30,4 +30,23 @@
             </actuator>
         </transmission>
+    </xacro:macro>
+    <xacro:macro name="sphere_marker" params="name markerX markerY markerZ markerRadius:=0.1">
+        <link name="${name}_marker">
+            <visual>
+                <origin xyz="0 0 0" rpy="0 0 0"/>
+                <geometry>
+                    <sphere radius="${markerRadius}"/>
+                </geometry>
+                <material name="orange"/>
+            </visual>
+        </link>
+        <gazebo reference="${name}_marker">
+            <material>Gazebo/Orange</material>
+        </gazebo>
+        <joint name="${name}_marker_joint" type="fixed">
+            <parent link="body"/>
+            <child link="${name}_marker"/>
+            <origin xyz="${x} ${y} ${z}" rpy="0 0 0"/>
+        </joint>
     </xacro:macro>
     <xacro:macro name="wing" params="name left">

File: urdf/planesil_model.xacro (robot description, xacro)
@@ -127,37 +127,16 @@
     </joint>
     <xacro:joint_transmission joint_name="propeller"/>
-    <link name="leftWingCP">
-        <visual>
-            <origin xyz="0 0 0" rpy="0 0 0"/>
-            <geometry>
-                <sphere radius="0.1"/>
-            </geometry>
-            <material name="orange"/>
-        </visual>
-    </link>
-    <gazebo reference="leftWingCP">
-        <material>Gazebo/Orange</material>
-    </gazebo>
-    <joint name="leftWingCP_joint" type="fixed">
-        <parent link="body"/>
-        <child link="leftWingCP"/>
-        <origin xyz="0 ${wingY/2} ${wingZ/2}" rpy="0 0 0"/>
-    </joint>
-    <link name="rightWingCP">
-        <visual>
-            <origin xyz="0 ${-wingY/2} ${wingZ/2}" rpy="0 0 0"/>
-            <geometry>
-                <sphere radius="0.1"/>
-            </geometry>
-            <material name="orange"/>
-        </visual>
-    </link>
-    <gazebo reference="rightWingCP">
-        <material>Gazebo/Orange</material>
-    </gazebo>
-    <joint name="rightWingCP_joint" type="fixed">
-        <parent link="base_link"/>
-        <child link="rightWingCP"/>
-    </joint>
+    <xacro:sphere_marker
+        name="leftWingCP"
+        markerX="0"
+        markerY="${wingY/2}"
+        markerZ="${wingZ/2}"
+    />
+    <xacro:sphere_marker
+        name="rightWingCP"
+        markerX="0"
+        markerY="${-wingY/2}"
+        markerZ="${wingZ/2}"
+    />
     <gazebo>
         <plugin name="propellerTopBlade" filename="libLiftDragPlugin.so">
