Commit message: Added elevator, removed counterweight, changed "aileron" to "controlsurface"

File: urdf/macros.xacro (robot description, xacro)
@@ -95,5 +95,5 @@
             <axis xyz="0 1 0" rpy="0 0 0"/>
         </joint>
-        <link name="${name}_aileron">
+        <link name="${name}_controlsurface">
             <inertial>
                 <origin xyz="0 0 0" rpy="0 0 0"/>
@@ -121,11 +121,11 @@
             </visual>
         </link>
-        <joint name="${name}_aileron_joint" type="continuous">
+        <joint name="${name}_controlsurface_joint" type="continuous">
             <parent link="${name}_wing" />
-            <child link="${name}_aileron" />
+            <child link="${name}_controlsurface" />
             <origin xyz="${-wingX/2 + -wingX/10} 0 0" rpy="0 0 0" />
             <axis xyz="0 1 0" rpy="0 0 0" />
         </joint>
-        <joint_transmission joint_name="${name}_aileron" reduction="100"/>
+        <joint_transmission joint_name="${name}_controlsurface" reduction="100"/>
     </xacro:macro>
     <xacro:macro name="landingGear" params="name front">

File: urdf/planesil_model.xacro (robot description, xacro)
@@ -3,28 +3,32 @@
     <xacro:include filename="$(find planesim_description)/urdf/materials.xacro" />
     <xacro:include filename="$(find planesim_description)/urdf/macros.xacro" />
-    <xacro:property name="PI" value="3.14"/>
-    <xacro:property name="bodyY" value="0.5"/>
-    <xacro:property name="bodyX" value="6"/>
-    <xacro:property name="bodyZ" value="0.5"/>
-    <xacro:property name="bodyMass" value="300"/>
-    <xacro:property name="wingY" value="5"/>
-    <xacro:property name="wingX" value="1"/>
-    <xacro:property name="wingZ" value="${bodyZ/4}"/>
-    <xacro:property name="wingMass" value="100"/>
-    <xacro:property name="landingGearY" value="${bodyY}"/>
-    <xacro:property name="landingGearX" value="0.125"/>
-    <xacro:property name="landingGearZ" value="1"/>
-    <xacro:property name="landingGearMass" value="10"/>
-    <xacro:property name="wheelWidth" value="0.1"/>
-    <xacro:property name="wheelRadius" value="0.25"/>
-    <xacro:property name="wheelMass" value="5"/>
-    <xacro:property name="propellerBlockX" value="0.25"/>
-    <xacro:property name="propellerBlockY" value="${bodyY/2}"/>
+    <xacro:property name="PI" value="3.14" />
+    <xacro:property name="bodyY" value="0.5" />
+    <xacro:property name="bodyX" value="6" />
+    <xacro:property name="bodyZ" value="0.5" />
+    <xacro:property name="bodyMass" value="300" />
+    <xacro:property name="wingY" value="5" />
+    <xacro:property name="wingX" value="1" />
+    <xacro:property name="wingZ" value="${bodyZ/4}" />
+    <xacro:property name="wingMass" value="100" />
+    <xacro:property name="landingGearY" value="${bodyY}" />
+    <xacro:property name="landingGearX" value="0.125" />
+    <xacro:property name="landingGearZ" value="1" />
+    <xacro:property name="landingGearMass" value="10" />
+    <xacro:property name="wheelWidth" value="0.1 "/>
+    <xacro:property name="wheelRadius" value="0.25 "/>
+    <xacro:property name="wheelMass" value="5" />
+    <xacro:property name="propellerBlockX" value="0.25" />
+    <xacro:property name="propellerBlockY" value="${bodyY/2}" />
     <xacro:property name="propellerBlockZ" value="${bodyZ/2}" />
-    <xacro:property name="propellerBlockMass" value="5"/>
-    <xacro:property name="propellerX" value="1.5"/>      <!-- Length of blade -->
-    <xacro:property name="propellerY" value="0.2"/>   <!-- Width of blade -->
-    <xacro:property name="propellerZ" value="0.1"/>    <!-- Thickness of blade -->
-    <xacro:property name="propellerMass" value="2"/>
+    <xacro:property name="propellerBlockMass" value="5" />
+    <xacro:property name="propellerX" value="1.5" />      <!-- Length of blade -->
+    <xacro:property name="propellerY" value="0.2" />   <!-- Width of blade -->
+    <xacro:property name="propellerZ" value="0.1" />    <!-- Thickness of blade -->
+    <xacro:property name="propellerMass" value="2" />
+    <xacro:property name="elevatorX" value="${wingX/2}" />
+    <xacro:property name="elevatorY" value="${bodyY*2}" />
+    <xacro:property name="elevatorZ" value="${bodyZ}" />
+    <xacro:property name="elevatorMass" value="40" />
     <!-- X axis is down the runway -->
     <!-- Y axis is to the left of the runway, looking down -->
@@ -127,4 +131,36 @@
     </joint>
     <xacro:joint_transmission joint_name="propeller"/>
+    <link name="elevator">
+        <inertial>
+            <origin xyz="0 0 0" rpy="0 0 0"/>
+                <mass value="${elevatorMass}"/>
+                <xacro:box_inertia m="${elevatorMass}" x="${elevatorX}" y="${elevatorY}" z="${elevatorZ}"/>
+            </inertial>
+            <collision>
+                <origin xyz="0 0 0" rpy="0 0 0"/>
+                <geometry>
+                    <box size="${elevatorX} ${elevatorY} ${elevatorZ}"/>
+                </geometry>
+            </collision>
+            <visual>
+                <origin xyz="0 0 0" rpy="0 0 0"/>
+                <geometry>
+                    <box size="${elevatorX} ${elevatorY} ${elevatorZ}"/>
+                </geometry>
+                <!-- Port/Starboard colors -->
+                <xacro:if value="${left == 1}">
+                    <material name="red"/>
+                </xacro:if>
+                <xacro:unless value="${left == 1}">
+                    <material name="green"/>
+                </xacro:unless>
+            </visual>
+    </link>
+    <joint name="elevator_joint" type="fixed">
+        <parent link="body" />
+        <child link="elevator" />
+        <origin xyz="${-bodyX/2} 0 0" rpy="0 0 0" />
+    </joint>
+    <!-- <joint_transmission joint_name="elevator_control" reduction="100"/> -->
     <xacro:sphere_marker
         name="leftWingCP"
@@ -187,5 +223,5 @@
             <upward> 0 0 1 </upward>
             <link_name>base_link</link_name>
-            <control_joint_name>left_aileron_joint</control_joint_name>
+            <control_joint_name>left_controlsurface_joint</control_joint_name>
             <control_joint_rad_to_cl>-2.0</control_joint_rad_to_cl>
         </plugin>
@@ -205,5 +241,5 @@
             <upward> 0 0 1 </upward>
             <link_name>base_link</link_name>
-            <control_joint_name>right_aileron_joint</control_joint_name>
+            <control_joint_name>right_controlsurface_joint</control_joint_name>
             <control_joint_rad_to_cl>-2.0</control_joint_rad_to_cl>
         </plugin>
@@ -219,34 +255,4 @@
         </controller:gazebo_ros_imu> -->
     </gazebo>
-    <xacro:property name="counterWeightCoGXOffset" value="${((propellerBlockMass * propellerBlockX/2) + propellerMass * (propellerBlockX/2 + propellerZ/2))
-                                                /(propellerBlockMass + propellerMass)}"/> <!-- Center of gravity from the edge of the body -->
-    <link name="counterWeight">
-        <inertial>
-            <origin xyz="0 0 0" rpy="0 0 0"/>
-            <mass value="${propellerBlockMass + propellerMass}"/>
-            <xacro:box_inertia m="${propellerBlockMass + propellerMass}" x="${2 * counterWeightCoGXOffset}" y="${bodyY}" z="${bodyZ}"/>
-        </inertial>
-        <collision>
-            <origin xyz="0 0 0" rpy="0 0 0"/>
-            <geometry>
-                <box size="${2 * counterWeightCoGXOffset} ${bodyY} ${bodyZ}"/>
-            </geometry>
-        </collision>
-        <visual>
-            <origin xyz="0 0 0" rpy="0 0 0"/>
-            <geometry>
-                <box size="${2 * counterWeightCoGXOffset} ${bodyY} ${bodyZ}"/>
-            </geometry>
-            <material name="orange"/>
-        </visual>
-    </link>
-    <gazebo reference="propellerBlock">
-        <material>Gazebo/Orange</material>
-    </gazebo>
-    <joint name="counterWeight_joint" type="fixed">
-        <parent link="body"/>
-        <child link="counterWeight"/>
-        <origin xyz="${-(bodyX/2 + counterWeightCoGXOffset)} 0 0" rpy="0 0 0"/>
-    </joint>
     <gazebo>
         <plugin name="gazebo_ros_control" filename="libgazebo_ros_control.so">

Commit message: Added elevator controlsurface

File: urdf/macros.xacro (robot description, xacro)
@@ -47,5 +47,5 @@
             <parent link="body"/>
             <child link="${name}_marker"/>
-            <origin xyz="${x} ${y} ${z}" rpy="0 0 0"/>
+            <origin xyz="${markerX} ${markerY} ${markerZ}" rpy="0 0 0"/>
         </joint>
     </xacro:macro>

File: urdf/planesil_model.xacro (robot description, xacro)
@@ -27,7 +27,7 @@
     <xacro:property name="propellerZ" value="0.1" />    <!-- Thickness of blade -->
     <xacro:property name="propellerMass" value="2" />
-    <xacro:property name="elevatorX" value="${wingX/2}" />
-    <xacro:property name="elevatorY" value="${bodyY*2}" />
-    <xacro:property name="elevatorZ" value="${bodyZ}" />
+    <xacro:property name="elevatorX" value="${wingX/3}" />
+    <xacro:property name="elevatorY" value="${bodyY*3}" />
+    <xacro:property name="elevatorZ" value="${wingZ}" />
     <xacro:property name="elevatorMass" value="40" />
     <!-- X axis is down the runway -->
@@ -148,19 +148,42 @@
                     <box size="${elevatorX} ${elevatorY} ${elevatorZ}"/>
                 </geometry>
-                <!-- Port/Starboard colors -->
-                <xacro:if value="${left == 1}">
-                    <material name="red"/>
-                </xacro:if>
-                <xacro:unless value="${left == 1}">
-                    <material name="green"/>
-                </xacro:unless>
+                <material name="blue"/>
             </visual>
     </link>
+    <gazebo reference="elevator">
+        <material>Gazebo/Blue</material>
+    </gazebo>
     <joint name="elevator_joint" type="fixed">
         <parent link="body" />
         <child link="elevator" />
-        <origin xyz="${-bodyX/2} 0 0" rpy="0 0 0" />
-    </joint>
-    <!-- <joint_transmission joint_name="elevator_control" reduction="100"/> -->
+        <origin xyz="${-bodyX/2 + -elevatorX/2} 0 0" rpy="0 0 0" />
+    </joint>
+    <link name="elevator_controlsurface">
+        <inertial>
+                <origin xyz="0 0 0" rpy="0 0 0"/>
+                <mass value="${elevatorMass/5}"/>
+                <xacro:box_inertia m="${elevatorMass/5}" x="${elevatorX/5}" y="${elevatorY}" z="${elevatorZ}"/>
+            </inertial>
+            <collision>
+                <origin xyz="0 0 0" rpy="0 0 0"/>
+                <geometry>
+                    <box size="${elevatorX/5} ${elevatorY} ${elevatorZ}"/>
+                </geometry>
+            </collision>
+            <visual>
+                <origin xyz="0 0 0" rpy="0 0 0"/>
+                <geometry>
+                    <box size="${elevatorX/5} ${elevatorY} ${elevatorZ}"/>
+                </geometry>
+                <material name="blue" />
+            </visual>
+    </link>
+    <joint name="elevator_controlsurface_joint" type="continuous">
+        <parent link="elevator" />
+        <child link="elevator_controlsurface" />
+        <origin xyz="${6 * -elevatorX/10} 0 0" rpy="0 0 0" />
+        <axis xyz="0 1 0" rpy="0 0 0" />
+    </joint>
+    <joint_transmission joint_name="elevator_controlsurface" reduction="100"/>
     <xacro:sphere_marker
         name="leftWingCP"
