Commit message: added right wing

File: urdf/planesil_model.xacro (robot description, xacro)
@@ -30,5 +30,5 @@
     <xacro:property name="wingY" value="5"/>
     <xacro:property name="wingX" value="1.5"/>
-    <xacro:property name="wingZ" value="${bodyZ/2}"/>
+    <xacro:property name="wingZ" value="${bodyZ/4}"/>
     <xacro:property name="wingMass" value="100"/>
     <!-- X axis is down the runway -->
@@ -92,4 +92,35 @@
         <axis xyz="0 1 0" rpy="0 0 0"/>
     </joint>
+    <link name="rightWing">
+        <inertial>
+            <origin xyz="0 0 0" rpy="0 0 0"/>
+            <mass value="${wingMass}"/>
+            <xacro:box_inertia m="${wingMass}" x="${wingX}" y="${wingY}" z="${wingZ}"/>
+        </inertial>
+        <collision>
+            <origin xyz="0 0 0" rpy="0 0 0"/>
+            <geometry>
+                <box size="${wingX} ${wingY} ${wingZ}"/>
+            </geometry>
+        </collision>
+        <visual>
+            <origin xyz="0 0 0" rpy="0 0 0"/>
+            <geometry>
+                <box size="${wingX} ${wingY} ${wingZ}"/>
+            </geometry>
+            <material name="green"/>
+        </visual>
+    </link>
+    <gazebo reference="rightWing">
+        <material>
+            Gazebo/Green
+        </material>
+    </gazebo>
+    <joint name="rightWing_joint" type="continuous">
+        <parent link="body"/>
+        <child link="rightWing"/>
+        <origin xyz="0 ${-(bodyY/2 + wingY/2)} 0" rpy="0 0 0"/>
+        <axis xyz="0 1 0" rpy="0 0 0"/>
+    </joint>
     <gazebo>
         <plugin name="gazebo_ros_control" filename="libgazebo_ros_control.so">

Commit message: Added counterweight

File: urdf/planesil_model.xacro (robot description, xacro)
@@ -89,5 +89,5 @@
         <material>Gazebo/Orange</material>
     </gazebo>
-    <joint name="propellorBlockJoint" type="fixed">
+    <joint name="propellorBlock_joint" type="fixed">
         <parent link="body"/>
         <child link="propellorBlock"/>
@@ -117,8 +117,38 @@
         <material>Gazebo/Blue</material>
     </gazebo>
-    <joint name="propellorJoint" type="continuous">
+    <joint name="propellor_joint" type="continuous">
         <parent link="propellorBlock" />
         <child link="propellor" />
         <origin xyz="${propellorBlockX/2 + propellorZ/2} 0 0" rpy="0 0 0"/>
+    </joint>
+    <xacro:property name="counterWeightCoGXOffset" value="${((propellorBlockMass * propellorBlockX/2) + propellorMass * (propellorBlockX/2 + propellorZ/2))
+                                                /(propellorBlockMass + propellorMass)}"/> <!-- Center of gravity from the edge of the body -->
+    <link name="counterWeight">
+        <inertial>
+            <origin xyz="0 0 0" rpy="0 0 0"/>
+            <mass value="${propellorBlockMass + propellorMass}"/>
+            <xacro:box_inertia m="${propellorBlockMass + propellorMass}" x="${2 * counterWeightCoGXOffset}" y="${bodyY}" z="${bodyZ}"/>
+        </inertial>
+        <collision>
+            <origin xyz="0 0 0" rpy="0 0 0"/>
+            <geometry>
+                <box size="${2 * counterWeightCoGXOffset} ${bodyY} ${bodyZ}"/>
+            </geometry>
+        </collision>
+        <visual>
+            <origin xyz="0 0 0" rpy="0 0 0"/>
+            <geometry>
+                <box size="${2 * counterWeightCoGXOffset} ${bodyY} ${bodyZ}"/>
+            </geometry>
+            <material name="orange"/>
+        </visual>
+    </link>
+    <gazebo reference="propellorBlock">
+        <material>Gazebo/Orange</material>
+    </gazebo>
+    <joint name="counterWeight_joint" type="fixed">
+        <parent link="body"/>
+        <child link="counterWeight"/>
+        <origin xyz="${-(bodyX/2 + counterWeightCoGXOffset)} 0 0" rpy="0 0 0"/>
     </joint>
     <gazebo>

Commit message: idk what I did but liftdrag works now for half the prop

File: urdf/planesil_model.xacro (robot description, xacro)
@@ -19,12 +19,12 @@
     <xacro:property name="wheelRadius" value="0.25"/>
     <xacro:property name="wheelMass" value="5"/>
-    <xacro:property name="propellorBlockX" value="0.25"/>
-    <xacro:property name="propellorBlockY" value="${bodyY/2}"/>
-    <xacro:property name="propellorBlockZ" value="${bodyZ/2}" />
-    <xacro:property name="propellorBlockMass" value="5"/>
-    <xacro:property name="propellorX" value="1.5"/>      <!-- Length of blade -->
-    <xacro:property name="propellorY" value="0.2"/>   <!-- Width of blade -->
-    <xacro:property name="propellorZ" value="0.1"/>    <!-- Thickness of blade -->
-    <xacro:property name="propellorMass" value="2"/>
+    <xacro:property name="propellerBlockX" value="0.25"/>
+    <xacro:property name="propellerBlockY" value="${bodyY/2}"/>
+    <xacro:property name="propellerBlockZ" value="${bodyZ/2}" />
+    <xacro:property name="propellerBlockMass" value="5"/>
+    <xacro:property name="propellerX" value="1.5"/>      <!-- Length of blade -->
+    <xacro:property name="propellerY" value="0.2"/>   <!-- Width of blade -->
+    <xacro:property name="propellerZ" value="0.1"/>    <!-- Thickness of blade -->
+    <xacro:property name="propellerMass" value="2"/>
     <!-- X axis is down the runway -->
     <!-- Y axis is to the left of the runway, looking down -->
@@ -66,14 +66,14 @@
     <xacro:wheel name="backLeft_wheel" front="-1" left="1" />
     <xacro:wheel name="backRight_wheel" front="-1" left="-1" />
-    <link name="propellorBlock">
+    <link name="propellerBlock">
         <inertial>
             <origin xyz="0 0 0" rpy="0 0 0"/>
-            <mass value="${propellorBlockMass}"/>
-            <xacro:box_inertia m="${propellorBlockMass}" x="${propellorBlockX}" y="${propellorBlockY}" z="${propellorBlockZ}"/>
+            <mass value="${propellerBlockMass}"/>
+            <xacro:box_inertia m="${propellerBlockMass}" x="${propellerBlockX}" y="${propellerBlockY}" z="${propellerBlockZ}"/>
         </inertial>
         <collision>
             <origin xyz="0 0 0" rpy="0 0 0"/>
             <geometry>
-                <box size="${propellorBlockX} ${propellorBlockY} ${propellorBlockZ}"/>
+                <box size="${propellerBlockX} ${propellerBlockY} ${propellerBlockZ}"/>
             </geometry>
         </collision>
@@ -81,27 +81,27 @@
             <origin xyz="0 0 0" rpy="0 0 0"/>
             <geometry>
-                <box size="${propellorBlockX} ${propellorBlockY} ${propellorBlockZ}"/>
+                <box size="${propellerBlockX} ${propellerBlockY} ${propellerBlockZ}"/>
             </geometry>
             <material name="orange"/>
         </visual>
     </link>
-    <gazebo reference="propellorBlock">
+    <gazebo reference="propellerBlock">
         <material>Gazebo/Orange</material>
     </gazebo>
-    <joint name="propellorBlock_joint" type="fixed">
+    <joint name="propellerBlock_joint" type="fixed">
         <parent link="body"/>
-        <child link="propellorBlock"/>
-        <origin xyz="${bodyX/2 + propellorBlockX/2} 0 0" rpy="0 0 0"/>
+        <child link="propellerBlock"/>
+        <origin xyz="${bodyX/2 + propellerBlockX/2} 0 0" rpy="0 0 0"/>
     </joint>
-    <link name="propellor">
+    <link name="propeller">
         <inertial>
             <origin xyz="0 0 0" rpy="0 ${PI/2} 0"/>
-            <mass value="${propellorMass}"/>
-            <xacro:box_inertia m="${propellorMass}" x="${propellorX}" y="${propellorY}" z="${propellorZ}"/>
+            <mass value="${propellerMass}"/>
+            <xacro:box_inertia m="${propellerMass}" x="${propellerX}" y="${propellerY}" z="${propellerZ}"/>
         </inertial>
         <collision>
             <origin xyz="0 0 0" rpy="0 ${PI/2} 0"/>
             <geometry>
-                <box size="${propellorX} ${propellorY} ${propellorZ}"/>
+                <box size="${propellerX} ${propellerY} ${propellerZ}"/>
             </geometry>
         </collision>
@@ -109,25 +109,63 @@
             <origin xyz="0 0 0" rpy="0 ${PI/2} 0"/>
             <geometry>
-                <box size="${propellorX} ${propellorY} ${propellorZ}"/>
+                <box size="${propellerX} ${propellerY} ${propellerZ}"/>
             </geometry>
             <material name="blue"/>
         </visual>
     </link>
-    <gazebo reference="propellor">
+    <gazebo reference="propeller">
         <material>Gazebo/Blue</material>
+        <kp>1000000</kp>
+        <kd>1000000</kd>
+        <mu1>10.0</mu1>
+        <mu2>10.0</mu2>
     </gazebo>
-    <joint name="propellor_joint" type="continuous">
-        <parent link="propellorBlock" />
-        <child link="propellor" />
-        <origin xyz="${propellorBlockX/2 + propellorZ/2} 0 0" rpy="0 0 0"/>
+    <joint name="propeller_joint" type="continuous">
+        <parent link="propellerBlock" />
+        <child link="propeller" />
+        <origin xyz="${propellerBlockX/2 + propellerZ/2} 0 0" rpy="0 0 0"/>
     </joint>
-    <xacro:joint_transmission name="propellor_transmission" joint_name="propellor_joint"/>
-    <xacro:property name="counterWeightCoGXOffset" value="${((propellorBlockMass * propellorBlockX/2) + propellorMass * (propellorBlockX/2 + propellorZ/2))
-                                                /(propellorBlockMass + propellorMass)}"/> <!-- Center of gravity from the edge of the body -->
+    <xacro:joint_transmission joint_name="propeller"/>
+    <gazebo>
+        <!-- <plugin name="propellerTopBlade" filename="libLiftDragPlugin.so">
+            <a0>0.4</a0>
+            <cla>4.752798721</cla>
+            <cda>0.6417112299</cda>
+            <cma>0</cma>
+            <alpha_stall>1.5</alpha_stall>
+            <cla_stall>-3.85</cla_stall>
+            <cda_stall>-0.9233984055</cda_stall>
+            <cma_stall>0</cma_stall>
+            <air_density>1.2041</air_density>
+            <cp> ${propellerZ/2} 0 ${propellerX/4} </cp>
+            <area>${propellerX * propellerY / 2}</area>
+            <forward> 0 1 0 </forward>
+            <upward> 1 0 0</upward>
+            <link_name>propeller</link_name>
+        </plugin> -->
+        <plugin name="propellerBottomBlade" filename="libLiftDragPlugin.so">
+            <a0>0.4</a0>
+            <cla>4.752798721</cla>
+            <cda>0.6417112299</cda>
+            <cma>0</cma>
+            <alpha_stall>1.5</alpha_stall>
+            <cla_stall>-3.85</cla_stall>
+            <cda_stall>-0.9233984055</cda_stall>
+            <cma_stall>0</cma_stall>
+            <air_density>1.2041</air_density>
+            <cp> ${propellerZ/2} 0 ${-propellerX/4} </cp>
+            <area>${propellerX * propellerY / 2}</area>
+            <forward> -1 0 0 </forward>
+            <upward> 0 0 1 </upward>
+            <link_name>propeller</link_name>
+        </plugin>
+    </gazebo>
+    <xacro:property name="counterWeightCoGXOffset" value="${((propellerBlockMass * propellerBlockX/2) + propellerMass * (propellerBlockX/2 + propellerZ/2))
+                                                /(propellerBlockMass + propellerMass)}"/> <!-- Center of gravity from the edge of the body -->
     <link name="counterWeight">
         <inertial>
             <origin xyz="0 0 0" rpy="0 0 0"/>
-            <mass value="${propellorBlockMass + propellorMass}"/>
-            <xacro:box_inertia m="${propellorBlockMass + propellorMass}" x="${2 * counterWeightCoGXOffset}" y="${bodyY}" z="${bodyZ}"/>
+            <mass value="${propellerBlockMass + propellerMass}"/>
+            <xacro:box_inertia m="${propellerBlockMass + propellerMass}" x="${2 * counterWeightCoGXOffset}" y="${bodyY}" z="${bodyZ}"/>
         </inertial>
         <collision>
@@ -145,5 +183,5 @@
         </visual>
     </link>
-    <gazebo reference="propellorBlock">
+    <gazebo reference="propellerBlock">
         <material>Gazebo/Orange</material>
     </gazebo>

Commit message: Made plane lighter, which can now take off. Still doesn't work; moving to gazebo sdf model

File: urdf/planesil_model.xacro (robot description, xacro)
@@ -7,9 +7,9 @@
     <xacro:property name="bodyX" value="6" />
     <xacro:property name="bodyZ" value="0.5" />
-    <xacro:property name="bodyMass" value="300" />
+    <xacro:property name="bodyMass" value="100" />
     <xacro:property name="wingY" value="5" />
     <xacro:property name="wingX" value="1" />
     <xacro:property name="wingZ" value="${bodyZ/4}" />
-    <xacro:property name="wingMass" value="100" />
+    <xacro:property name="wingMass" value="50" />
     <xacro:property name="landingGearY" value="${bodyY}" />
     <xacro:property name="landingGearX" value="0.125" />
@@ -28,7 +28,7 @@
     <xacro:property name="propellerMass" value="2" />
     <xacro:property name="elevatorX" value="${wingX/3}" />
-    <xacro:property name="elevatorY" value="${bodyY*3}" />
+    <xacro:property name="elevatorY" value="${wingY/2}" />
     <xacro:property name="elevatorZ" value="${wingZ}" />
-    <xacro:property name="elevatorMass" value="40" />
+    <xacro:property name="elevatorMass" value="125" />
     <!-- X axis is down the runway -->
     <!-- Y axis is to the left of the runway, looking down -->
@@ -157,30 +157,30 @@
         <parent link="body" />
         <child link="elevator" />
-        <origin xyz="${-bodyX/2 + -elevatorX/2} 0 0" rpy="0 0 0" />
+        <origin xyz="${-bodyX/2 + elevatorX/2} 0 0" rpy="0 0 0" />
     </joint>
     <link name="elevator_controlsurface">
         <inertial>
-                <origin xyz="0 0 0" rpy="0 0 0"/>
-                <mass value="${elevatorMass/5}"/>
-                <xacro:box_inertia m="${elevatorMass/5}" x="${elevatorX/5}" y="${elevatorY}" z="${elevatorZ}"/>
-            </inertial>
-            <collision>
-                <origin xyz="0 0 0" rpy="0 0 0"/>
-                <geometry>
+            <origin xyz="${-elevatorX/10} 0 0" rpy="0 0 0"/>
+            <mass value="${elevatorMass/5}"/>
+            <xacro:box_inertia m="${elevatorMass/5}" x="${elevatorX/3}" y="${elevatorY}" z="${elevatorZ/2}"/>
+        </inertial>
+        <collision>
+            <origin xyz="${-elevatorX/10} 0 0" rpy="0 0 0"/>
+            <geometry>
                     <box size="${elevatorX/5} ${elevatorY} ${elevatorZ}"/>
-                </geometry>
-            </collision>
-            <visual>
-                <origin xyz="0 0 0" rpy="0 0 0"/>
-                <geometry>
-                    <box size="${elevatorX/5} ${elevatorY} ${elevatorZ}"/>
-                </geometry>
-                <material name="blue" />
-            </visual>
+            </geometry>
+        </collision>
+        <visual>
+            <origin xyz="${-elevatorX/10} 0 0" rpy="0 0 0"/>
+            <geometry>
+                <box size="${-elevatorX/3} ${elevatorY} ${elevatorZ/2}"/>
+            </geometry>
+            <material name="blue" />
+        </visual>
     </link>
     <joint name="elevator_controlsurface_joint" type="continuous">
         <parent link="elevator" />
         <child link="elevator_controlsurface" />
-        <origin xyz="${6 * -elevatorX/10} 0 0" rpy="0 0 0" />
+        <origin xyz="${-elevatorX/2} 0 0" rpy="0 0 0" />
         <axis xyz="0 1 0" rpy="0 0 0" />
     </joint>
@@ -198,4 +198,10 @@
         markerZ="${wingZ/2}"
     />
+    <xacro:sphere_marker
+        name="elevatorCP"
+        markerX="${-bodyX/2 + -elevatorX/2}"
+        markerY="0"
+        markerZ="${elevatorZ/2}"
+    />
     <gazebo>
         <plugin name="propellerTopBlade" filename="libLiftDragPlugin.so">
@@ -208,5 +214,5 @@
             <cda_stall>-0.9233984055</cda_stall>
             <cma_stall>0</cma_stall>
-            <air_density>1.2041</air_density>
+            <air_density>1</air_density>
             <cp> ${propellerZ/2} 0 ${propellerX/4} </cp>
             <area>${propellerX * propellerY / 2}</area>
@@ -224,5 +230,5 @@
             <cda_stall>-0.9233984055</cda_stall>
             <cma_stall>0</cma_stall>
-            <air_density>1.2041</air_density>
+            <air_density>1</air_density>
             <cp> ${propellerZ/2} 0 ${-propellerX/4} </cp>
             <area> 0.5 </area>
@@ -240,5 +246,5 @@
             <cda_stall>-0.9233984055</cda_stall>
             <cma_stall>0</cma_stall>
-            <air_density> 1.2041 </air_density>
+            <air_density> 2 </air_density>
             <cp> 0 ${wingY/2} ${wingZ/2}</cp>
             <area> ${(wingX/2) * (wingY/2)}</area>
@@ -258,5 +264,5 @@
             <cda_stall>-0.9233984055</cda_stall>
             <cma_stall>0</cma_stall>
-            <air_density> 1.2041 </air_density>
+            <air_density> 2 </air_density>
             <cp> 0 ${-wingY/2} ${wingZ/2}</cp>
             <area> ${(wingX/2) * (wingY/2)}</area>
@@ -267,14 +273,32 @@
             <control_joint_rad_to_cl>-2.0</control_joint_rad_to_cl>
         </plugin>
-        <!-- <controller:gazebo_ros_imu name="imu_controller" plugin="libgazebo_ros_imu.so">
-            <alwaysOn>true</alwaysOn>
-            <updateRate>50.0</updateRate>
-            <bodyName>body</bodyName>
-            <topicName>imu_data</topicName>
-            <gaussianNoise>2.89e-08</gaussianNoise>
-            <xyzOffsets>0 0 0</xyzOffsets>
-            <rpyOffsets>0 0 0</rpyOffsets>
-            <interface:position name="imu_position"/>
-        </controller:gazebo_ros_imu> -->
+        <plugin name="elevator" filename="libplanesim_liftdrag.so">
+            <a0>0.05984281113</a0>
+            <cla>4.752798721</cla>
+            <cda>0.6417112299</cda>
+            <cma>-1.8</cma>
+            <alpha_stall>0.3391428111</alpha_stall>
+            <cla_stall>-3.85</cla_stall>
+            <cda_stall>-0.9233984055</cda_stall>
+            <cma_stall>0</cma_stall>
+            <air_density> 2 </air_density>
+            <cp> ${-bodyX/2 + -elevatorX/2} 0 ${elevatorZ/2}</cp>
+            <area> ${(elevatorX/2) * (elevatorY/2)}</area>
+            <forward> 1 0 0 </forward>
+            <upward> 0 0 1 </upward>
+            <link_name>base_link</link_name>
+            <control_joint_name>elevator_controlsurface_joint</control_joint_name>
+            <control_joint_rad_to_cl>-2.0</control_joint_rad_to_cl>
+        </plugin>
+        <!-- <plugin name="ForceTester_left" filename="libgazebo_forcetest_plugin.so">
+            <name>left_wing</name>
+            <targetPoint>0 ${wingY/2} 0</targetPoint>
+            <link_name>base_link</link_name>
+        </plugin>
+        <plugin name="ForceTester_right" filename="libgazebo_forcetest_plugin.so">
+            <name>right_wing</name>
+            <targetPoint>0 ${-wingY/2} 0</targetPoint>
+            <link_name>base_link</link_name>
+        </plugin> -->
     </gazebo>
     <gazebo>
